File: cypher_matrix.sch (KiCad schematic (older format))
At the start: 272 parts

Commit message: Update files to rev. 2
correction of error in the crystal wiring

adjusted all the diode footprints to be easier to read

moved D70 to be vertical and placed more in line with the rest of the diodes

bumped silkscreen to rev. 2
Parts:
- D10, D11, D12, D13, D14, D15, D16, D17, D18, D19, D21, D22, D23, D24, D25, D26, D27, D28, D29, D30, D31, D32, D33, D34, D35, D36, D37, D38, D39, D4, D40, D41, D42, D43, D44, D45, D46, D47, D48, D49, D5, D50, D51, D52, D53, D54, D55, D56, D57, D58, D59, D6, D60, D61, D62, D63, D64, D65, D66, D67, D68, D69, D7, D70, D71, D72, D73, D74, D75, D76, D77, D78, D79, D8, D80, D81, D82, D83, D84, D85, D86, D87, D88, D89, D9, D90: value D_Small -> 1N4148
- R10, R11, R12, R13, R14, R15, R16, R17, R18, R19, R20, R21, R22, R23, R24, R25, R26, R27, R29, R30, R31, R32, R33, R34, R35, R36, R37, R38, R39, R40, R41, R42, R43, R44, R45, R46, R47, R48, R49, R50, R51, R52, R53, R54, R55, R56, R57, R58, R59, R60, R61, R62, R63, R64, R65, R66, R67, R68, R69, R70, R71, R72, R73, R74, R75, R76, R77, R78, R79, R80, R81, R82, R83, R84, R85, R86, R87, R88, R89, R9, R90, R91, R92, R93, R94, R95: value 1K -> 470

Commit message: update to rev5
Parts:
- added D20, D92: 1N4148, Diode_SMD:D_0603_1608Metric, symbol Device:D_Small
- added MX101: Split_left, 19mmMX:MXOnly-2.75U-FLIPPED-ReversedStabilizers, symbol MX_Alps_Hybrid:MX-LED
- added MX102: Split_left, MX_Only:MXOnly-2.25U-ReversedStabilizers, symbol MX_Alps_Hybrid:MX-LED
- added MX103: Split_center, MX_Only:MXOnly-1.25U, symbol MX_Alps_Hybrid:MX-LED
- added MX104: Split_center, 19mmMX:MXOnly-1.25U-FLIPPED, symbol MX_Alps_Hybrid:MX-LED
- added MX105: Split_right, MX_Only:MXOnly-2.25U-ReversedStabilizers, symbol MX_Alps_Hybrid:MX-LED
- added MX106: Split_right, 19mmMX:MXOnly-2.75U-FLIPPED-ReversedStabilizers, symbol MX_Alps_Hybrid:MX-LED
- added R97, R99: 470, Resistor_SMD:R_0603_1608Metric, symbol Device:R_Small
- D10, D11, D12, D13, D14, D15, D16, D17, D18, D19, D21, D22, D23, D24, D25, D26, D27, D28, D29, D30, D31, D32, D33, D34, D35, D36, D37, D38, D39, D4, D40, D41, D42, D43, D44, D45, D46, D47, D48, D49, D5, D50, D51, D52, D53, D54, D55, D56, D57, D58, D59, D6, D60, D61, D62, D63, D64, D65, D66, D67, D68, D69, D7, D70, D71, D72, D73, D74, D75, D76, D77, D78, D79, D8, D80, D81, D82, D83, D84, D85, D86, D87, D88, D89, D9, D90: footprint Diode_SMD:D_0805_2012Metric_Pad1.15x1.40mm_HandSolder -> Diode_SMD:D_0603_1608Metric
- MX1, MX75: footprint MX_Alps_Hybrid:MXOnly-2.25U -> MX_Only:MXOnly-2.25U; symbol MX_Alps_Hybrids:MX-1U -> MX_Alps_Hybrid:MX-LED
- MX10, MX11, MX12, MX13, MX14, MX16, MX17, MX18, MX19, MX21, MX22, MX23, MX24, MX26, MX27, MX28, MX29, MX30, MX31, MX32, MX33, MX36, MX37, MX38, MX39, MX4, MX41, MX42, MX43, MX44, MX45, MX46, MX47, MX48, MX49, MX50, MX51, MX52, MX55, MX56, MX57, MX58, MX59, MX61, MX62, MX63, MX64, MX66, MX67, MX68, MX70, MX71, MX76, MX77, MX78, MX79, MX80, MX81, MX82, MX83, MX84, MX85, MX86, MX87, MX88, MX89, MX90, MX91, MX92, MX93, MX94, MX95, MX96, MX97, MX99: footprint MX_Alps_Hybrid:MXOnly-1U -> MX_Only:MXOnly-1U; symbol MX_Alps_Hybrids:MX-1U -> MX_Alps_Hybrid:MX-LED
- MX100, MX98: footprint MX_Alps_Hybrid:MXOnly-2U-ReversedStabilizers -> MX_Only:MXOnly-2U-ReversedStabilizers; symbol MX_Alps_Hybrids:MX-1U -> MX_Alps_Hybrid:MX-LED
- MX15, MX5, MX54, MX60, MX74: footprint MX_Alps_Hybrid:MXOnly-1.5U -> MX_Only:MXOnly-1.5U; symbol MX_Alps_Hybrids:MX-1U -> MX_Alps_Hybrid:MX-LED
- MX2: footprint MX_Alps_Hybrid:MXOnly-1.5U-FLIPPED -> MX_Only:MXOnly-1.5U-FLIPPED; symbol MX_Alps_Hybrids:MX-1U -> MX_Alps_Hybrid:MX-LED
- MX20, MX3, MX53, MX7, MX8: footprint MX_Alps_Hybrid:MXOnly-1.25U -> MX_Only:MXOnly-1.25U; symbol MX_Alps_Hybrids:MX-1U -> MX_Alps_Hybrid:MX-LED
- MX25, MX65: footprint MX_Alps_Hybrid:MXOnly-1.25U-FLIPPED -> MX_Only:MXOnly-1.25U-FLIPPED; symbol MX_Alps_Hybrids:MX-1U -> MX_Alps_Hybrid:MX-LED
- MX34: footprint MX_Alps_Hybrid:MXOnly-6.25U-FLIPPED-ReversedStabilizers -> MX_Only:MXOnly-6.25U-FLIPPED-ReversedStabilizers; symbol MX_Alps_Hybrids:MX-1U -> MX_Alps_Hybrid:MX-LED
- MX35: footprint MX_Alps_Hybrid:MXOnly-7U-ReversedStabilizers -> 19mmMX:MXOnly-7U-FLIPPED-ReversedStabilizers; symbol MX_Alps_Hybrids:MX-1U -> MX_Alps_Hybrid:MX-LED
- MX40: footprint MX_Alps_Hybrid:MXOnly-6U-ReversedStabilizers -> MX_Only:MXOnly-6U-ReversedStabilizers; symbol MX_Alps_Hybrids:MX-1U -> MX_Alps_Hybrid:MX-LED
- MX6: footprint MX_Alps_Hybrid:MXOnly-1.75U-FLIPPED -> MX_Only:MXOnly-1.75U-FLIPPED; symbol MX_Alps_Hybrids:MX-1U -> MX_Alps_Hybrid:MX-LED
- MX69: footprint MX_Alps_Hybrid:MXOnly-1.75U -> MX_Only:MXOnly-1.75U; symbol MX_Alps_Hybrids:MX-1U -> MX_Alps_Hybrid:MX-LED
- MX72: footprint MX_Alps_Hybrid:MXOnly-ISO-ROTATED-ReversedStabilizers -> MX_Only:MXOnly-ISO-ReversedStabilizers; symbol MX_Alps_Hybrids:MX-1U -> MX_Alps_Hybrid:MX-LED
- MX73: footprint MX_Alps_Hybrid:MXOnly-2U -> MX_Only:MXOnly-2U; symbol MX_Alps_Hybrids:MX-1U -> MX_Alps_Hybrid:MX-LED
- MX9: footprint MX_Alps_Hybrid:MXOnly-1.25U-FLIPPED -> MX_Only:MXOnly-1U-FLIPPED; symbol MX_Alps_Hybrids:MX-1U -> MX_Alps_Hybrid:MX-LED
- R10, R11, R12, R13, R14, R15, R16, R17, R18, R19, R20, R21, R22, R23, R24, R25, R26, R27, R29, R30, R31, R32, R33, R34, R35, R36, R37, R38, R39, R40, R41, R42, R43, R44, R45, R46, R47, R48, R49, R50, R51, R52, R53, R54, R55, R56, R57, R58, R59, R60, R61, R62, R63, R64, R65, R66, R67, R68, R69, R70, R71, R72, R73, R74, R75, R76, R77, R78, R79, R80, R81, R82, R83, R84, R85, R86, R87, R88, R89, R9, R90, R91, R92, R93, R94, R95: footprint Resistor_SMD:R_0805_2012Metric_Pad1.15x1.40mm_HandSolder -> Resistor_SMD:R_0603_1608Metric
Connections:
- wire segments 1155 -> 1227
Other:
- moved on the sheet: D5
