File: cypher_matrix.sch (KiCad schematic (older format))
At the start: 282 parts

Commit message: Added base for Rev 6
Connections:
- net Row5 is gone; now on net Row0: D51.1 (K), D56.1 (K), D63.1 (K), D65.1 (K), D70.1 (K), D71.1 (K), D77.1 (K), D84.1 (K), D87.1 (K)
- net Row6 is gone; now on net Row1: D53.1 (K), D57.1 (K), D61.1 (K), D69.1 (K), D73.1 (K), D78.1 (K), D81.1 (K), D88.1 (K)
- net Row7 is gone; now on net Row2: D52.1 (K), D58.1 (K), D64.1 (K), D66.1 (K), D72.1 (K), D76.1 (K), D82.1 (K), D89.1 (K)
- net Row8 is gone; now on net Row3: D54.1 (K), D59.1 (K), D62.1 (K), D67.1 (K), D74.1 (K), D79.1 (K), D85.1 (K), D90.1 (K)
- net Row9 is gone; now on net Row4: D50.1 (K), D55.1 (K), D60.1 (K), D68.1 (K), D75.1 (K), D80.1 (K), D83.1 (K), D86.1 (K)
- net Col0: no longer MX54.1 (COL), MX55.1 (COL), MX56.1 (COL), MX57.1 (COL), MX58.1 (COL), MX59.1 (COL)
- net Col1: no longer MX60.1 (COL), MX61.1 (COL), MX62.1 (COL), MX63.1 (COL), MX64.1 (COL), MX65.1 (COL)
- net Col2: no longer MX66.1 (COL), MX67.1 (COL), MX68.1 (COL), MX69.1 (COL), MX70.1 (COL)
- net Col3: no longer MX71.1 (COL), MX72.1 (COL), MX73.1 (COL), MX74.1 (COL), MX75.1 (COL), MX76.1 (COL), MX77.1 (COL)
- net Col4: no longer MX78.1 (COL)
- net Col5: no longer MX79.1 (COL), MX80.1 (COL), MX81.1 (COL), MX82.1 (COL), MX83.1 (COL)
- net Col6: no longer MX84.1 (COL), MX85.1 (COL), MX86.1 (COL), MX87.1 (COL), MX88.1 (COL)
- net Col7: no longer MX89.1 (COL), MX90.1 (COL), MX91.1 (COL), MX92.1 (COL), MX93.1 (COL)
- net Col8: no longer MX100.1 (COL), MX94.1 (COL), MX95.1 (COL), MX96.1 (COL), MX97.1 (COL), MX98.1 (COL), MX99.1 (COL)
- new net Col10: MX54.1 (COL), MX55.1 (COL), MX56.1 (COL), MX57.1 (COL), MX58.1 (COL), MX59.1 (COL)
- new net Col11: MX60.1 (COL), MX61.1 (COL), MX62.1 (COL), MX63.1 (COL), MX64.1 (COL), MX65.1 (COL)
- new net Col12: MX66.1 (COL), MX67.1 (COL), MX68.1 (COL), MX69.1 (COL), MX70.1 (COL)
- new net Col13: MX71.1 (COL), MX72.1 (COL), MX73.1 (COL), MX74.1 (COL), MX75.1 (COL), MX76.1 (COL), MX77.1 (COL)
- new net Col14: MX78.1 (COL)
- new net Col15: MX79.1 (COL), MX80.1 (COL), MX81.1 (COL), MX82.1 (COL), MX83.1 (COL)
- new net Col16: MX84.1 (COL), MX85.1 (COL), MX86.1 (COL), MX87.1 (COL), MX88.1 (COL)
- new net Col17: MX89.1 (COL), MX90.1 (COL), MX91.1 (COL), MX92.1 (COL), MX93.1 (COL)
- new net Col18: MX100.1 (COL), MX94.1 (COL), MX95.1 (COL), MX96.1 (COL), MX97.1 (COL), MX98.1 (COL), MX99.1 (COL)
Other:
- moved on the sheet: D10, D13, D17, D18, D19, D23, D26, D27, D28, D31, D33, D36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

Commit message: updated rev6
Parts:
- D10, D11, D12, D13, D14, D15, D16, D17, D18, D19, D20, D21, D22, D23, D24, D25, D26, D27, D28, D29, D30, D31, D32, D33, D34, D35, D36, D37, D38, D39, D4, D40, D41, D42, D43, D44, D45, D46, D47, D48, D49, D5, D50, D51, D52, D53, D54, D55, D56, D57, D58, D59, D6, D60, D61, D62, D63, D64, D65, D66, D67, D68, D69, D7, D70, D71, D72, D73, D74, D75, D76, D77, D78, D79, D8, D80, D81, D82, D83, D84, D85, D86, D87, D88, D89, D9, D90, D92: footprint Diode_SMD:D_0603_1608Metric -> Diode_SMD:D_SOD-123
