File: cypher.kicad_pcb (KiCad board)
At the start: 2 copper layers, 370.1 x 106 mm, 313 parts, among them J2 AVR-ISP-6, J3 Breakout, Q1 MMBT3904, SW1 SW_Push, U1 ATmega32U4-MU, U2 PRTR5V0U2X, Y1 16Mhz

Commit message: Added base for Rev 6
Parts:
- removed C8: 1uf, Capacitor_SMD:C_0603_1608Metric
- removed J2: AVR-ISP-6, Connector_PinHeader_2.54mm:PinHeader_2x03_P2.54mm_Vertical
- removed R3: 10k, Resistor_SMD:R_0603_1608Metric
- removed R4: 10K, Resistor_SMD:R_0603_1608Metric
- removed R6, R7, R8: 470, Resistor_SMD:R_0603_1608Metric
- removed Y1: 16Mhz, Crystal:Crystal_SMD_2520-4Pin_2.5x2.0mm
- removed svg2mod: G***, Artwork:CableCarLogo
- added D91: D, Diode_SMD:D_0603_1608Metric, B.Cu at (284.4, 183.1)
- added Q2: MMBT3904, Package_TO_SOT_SMD:SOT-23, B.Cu at (314.5, 127.1)
- added U3: LD3985G33R_TSOT23, Package_TO_SOT_SMD:TSOT-23-5, B.Cu at (317.3, 144.6)
- C2: value 22pF -> 10nf
- C3: value 22pF -> 10uf
- C4: value 100nF -> 4.7uf
- D1: value CAPS -> WS2812B; footprint LED_THT:LED_D1.8mm_W3.3mm_H2.4mm -> CrumpPrints:WS2812-2020
- D2: value Num -> WS2812B; footprint LED_THT:LED_D1.8mm_W3.3mm_H2.4mm -> CrumpPrints:WS2812-2020
- D3: value Scroll -> WS2812B; footprint LED_THT:LED_D1.8mm_W3.3mm_H2.4mm -> CrumpPrints:WS2812-2020
- F1: footprint Fuse:Fuse_0805_2012Metric -> Fuse:Fuse_0603_1608Metric
- Q1: value MMBT3904 -> BC850
- R1: value 22R -> 1.5k
- R2: value 22R -> 30k
- SW1: footprint Connector_PinHeader_2.54mm:PinHeader_2x01_P2.54mm_Vertical -> reset:ResetShort
- U1: value ATmega32U4-MU -> STM32F072CBTx; footprint Package_DFN_QFN:QFN-44-1EP_7x7mm_P0.5mm_EP5.2x5.2mm -> Package_QFP:LQFP-48_7x7mm_P0.5mm
- U2: footprint PRTR5V0U2X:SOT143B -> random-keyboard-parts:SOT143B
- moved R1 96.9 mm to (284.4, 186.0), turned to 0 degrees
- moved R2 91.4 mm to (284.4, 180.1), turned to 180 degrees
- moved SW1 68.2 mm to (172.6, 193.6)
- moved Q1 63.8 mm to (288.8, 185.5), turned to 0 degrees
- moved J3 56.7 mm to (315.9, 133.7)
- moved C3 40.3 mm to (288.1, 180.1), turned to 180 degrees
- moved C1 18.0 mm to (313.3, 144.6), turned to 90 degrees
- moved C2 12.5 mm to (321.7, 144.5), turned to 270 degrees
- moved C6 11.5 mm to (323.3, 168.0), turned to 45 degrees
- moved C4 9.57 mm to (322.5, 159.5), turned to 315 degrees
- moved C5 4.86 mm to (319.2, 171.8)
- moved D1 1.29 mm to (315.8, 113.2)
- moved U1 1.27 mm to (314.4, 165.0), turned to 135 degrees
- moved D2 1.23 mm to (315.7, 116.4)
- moved D3 1.23 mm to (315.7, 119.5)
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Connections:
- C2 pad 1: XTAL1 -> Net-(C2-Pad1)
- C3 pad 1: XTAL2 -> BOOT0
- C4 pad 2: +5V -> +3V3
- C5 pad 2: +5V -> +3V3
- C6 pad 2: +5V -> +3V3
- C7 pad 2: +5V -> +3V3
- D1 pad 1: Net-(D1-Pad1) -> +5V
- D1 pad 2: Caps -> B15
- D2 pad 1: Net-(D2-Pad1) -> +5V
- D2 pad 2: Num -> Net-(D1-Pad4)
- D3 pad 1: Net-(D3-Pad1) -> +5V
- D3 pad 2: Scrl -> Net-(D2-Pad4)
- D50 pad 1: Row9 -> Row4
- D51 pad 1: Row5 -> Row0
- D52 pad 1: Row7 -> Row2
- D53 pad 1: Row6 -> Row1
- D54 pad 1: Row8 -> Row3
- D55 pad 1: Row9 -> Row4
- D56 pad 1: Row5 -> Row0
- D57 pad 1: Row6 -> Row1
- D58 pad 1: Row7 -> Row2
- D59 pad 1: Row8 -> Row3
- D60 pad 1: Row9 -> Row4
- D61 pad 1: Row6 -> Row1
- D62 pad 1: Row8 -> Row3
- D63 pad 1: Row5 -> Row0
- D64 pad 1: Row7 -> Row2
- D65 pad 1: Row5 -> Row0
- D66 pad 1: Row7 -> Row2
- D67 pad 1: Row8 -> Row3
- D68 pad 1: Row9 -> Row4
- D69 pad 1: Row6 -> Row1
- D70 pad 1: Row5 -> Row0
- D71 pad 1: Row5 -> Row0
- D72 pad 1: Row7 -> Row2
- D73 pad 1: Row6 -> Row1
- D74 pad 1: Row8 -> Row3
- D75 pad 1: Row9 -> Row4
- D76 pad 1: Row7 -> Row2
- D77 pad 1: Row5 -> Row0
- D78 pad 1: Row6 -> Row1
- D79 pad 1: Row8 -> Row3
- D80 pad 1: Row9 -> Row4
- D81 pad 1: Row6 -> Row1
- D82 pad 1: Row7 -> Row2
- D83 pad 1: Row9 -> Row4
- D84 pad 1: Row5 -> Row0
- D85 pad 1: Row8 -> Row3
- D86 pad 1: Row9 -> Row4
- D87 pad 1: Row5 -> Row0
- D88 pad 1: Row6 -> Row1
- D89 pad 1: Row7 -> Row2
- D90 pad 1: Row8 -> Row3
- J3 pad 1: E6 -> B15
- MX100 pad 1: Col8 -> Col18
- MX54 pad 1: Col0 -> Col10
- MX55 pad 1: Col0 -> Col10
- MX56 pad 1: Col0 -> Col10
- MX57 pad 1: Col0 -> Col10
- MX58 pad 1: Col0 -> Col10
- MX59 pad 1: Col0 -> Col10
- MX60 pad 1: Col1 -> Col11
- MX61 pad 1: Col1 -> Col11
- MX62 pad 1: Col1 -> Col11
- MX63 pad 1: Col1 -> Col11
- MX64 pad 1: Col1 -> Col11
- MX65 pad 1: Col1 -> Col11
- MX66 pad 1: Col2 -> Col12
- MX67 pad 1: Col2 -> Col12
- MX68 pad 1: Col2 -> Col12
- MX69 pad 1: Col2 -> Col12
- MX70 pad 1: Col2 -> Col12
- MX71 pad 1: Col3 -> Col13
- MX72 pad 1: Col3 -> Col13
- MX73 pad 1: Col3 -> Col13
- MX74 pad 1: Col3 -> Col13
- MX75 pad 1: Col3 -> Col13
- MX76 pad 1: Col3 -> Col13
- MX77 pad 1: Col3 -> Col13
- MX78 pad 1: Col4 -> Col14
- MX79 pad 1: Col5 -> Col15
- MX80 pad 1: Col5 -> Col15
- MX81 pad 1: Col5 -> Col15
- MX82 pad 1: Col5 -> Col15
- MX83 pad 1: Col5 -> Col15
- MX84 pad 1: Col6 -> Col16
- MX85 pad 1: Col6 -> Col16
- MX86 pad 1: Col6 -> Col16
- MX87 pad 1: Col6 -> Col16
- MX88 pad 1: Col6 -> Col16
- MX89 pad 1: Col7 -> Col17
- MX90 pad 1: Col7 -> Col17
- MX91 pad 1: Col7 -> Col17
- MX92 pad 1: Col7 -> Col17
- MX93 pad 1: Col7 -> Col17
- MX94 pad 1: Col8 -> Col18
- MX95 pad 1: Col8 -> Col18
- MX96 pad 1: Col8 -> Col18
- MX97 pad 1: Col8 -> Col18
- MX98 pad 1: Col8 -> Col18
- MX99 pad 1: Col8 -> Col18
- Q1 pad 3: LEDGND -> NRST
- R1 pad 1: D- -> Net-(D91-Pad2)
- R1 pad 2: Net-(R1-Pad2) -> Net-(Q1-Pad1)
- R2 pad 1: D+ -> BOOT0
- R2 pad 2: Net-(R2-Pad2) -> GND
- R5 pad 1: Net-(Q1-Pad1) -> Net-(Q2-Pad1)
- SW1 pad 1: GND -> +3V3
- SW1 pad 2: RESET -> Net-(D91-Pad2)
- U1 pad 1: E6 -> +3V3
- U1 pad 10: Col7 -> Net-(U1-Pad10)
- U1 pad 11: Col6 -> Col13
- U1 pad 12: Col5 -> Col12
- U1 pad 13: RESET -> Col11
- U1 pad 14: +5V -> Col10
- U1 pad 15: GND -> Col9
- U1 pad 16: XTAL2 -> Net-(R5-Pad2)
- U1 pad 17: XTAL1 -> Net-(U1-Pad17)
- U1 pad 18: Net-(R5-Pad2) -> Col8
- U1 pad 19: Row5 -> Col7
- U1 pad 2: +5V -> Col16
- U1 pad 20: Scrl -> Col6
- U1 pad 21: Num -> Row4
- U1 pad 22: Caps -> Row3
- U1 pad 24: +5V -> +3V3
- U1 pad 25: Row7 -> Col5
- U1 pad 26: Col0 -> Col4
- U1 pad 27: Col1 -> Col3
- U1 pad 28: Col2 -> LED_OUT
- U1 pad 29: Col3 -> Col2
- U1 pad 3: D- -> Col17
- U1 pad 30: Col4 -> Col1
- U1 pad 31: Row8 -> Col0
- U1 pad 32: Row9 -> D-
- U1 pad 33: Net-(R4-Pad2) -> D+
- U1 pad 34: +5V -> Col14
- U1 pad 36: Row4 -> +3V3
- U1 pad 37: Row3 -> Row0
- U1 pad 38: Row2 -> Row1
- U1 pad 39: Row6 -> Row2
- U1 pad 4: D+ -> Col15
- U1 pad 40: Row1 -> Net-(U1-Pad40)
- U1 pad 41: Col9 -> Net-(U1-Pad41)
- U1 pad 43: GND -> Net-(U1-Pad43)
- U1 pad 44: +5V -> BOOT0
- U1 pad 45: GND -> Net-(U1-Pad45)
- U1 pad 5: GND -> Net-(U1-Pad5)
- U1 pad 7: +5V -> NRST
- U1 pad 8: Row0 -> GND
- U1 pad 9: Col8 -> +3V3
- U2 pad 2: Net-(R1-Pad2) -> D+
- U2 pad 3: Net-(R2-Pad2) -> D-
- USB1 pad 5: Net-(R1-Pad2) -> D-
- USB1 pad 6: Net-(R2-Pad2) -> D+
- USB1 pad 7: Net-(R1-Pad2) -> D-
- USB1 pad 8: Net-(R2-Pad2) -> D+
Routing:
- net RESET: track 312.7 -> 0.00 mm, vias 1 -> 0
- net Row5: track 246.0 -> 0.00 mm, vias 4 -> 0
- net Col7: track 496.9 -> 254.1 mm, vias 8 -> 0
- net +3V3: track 0.00 -> 242.4 mm, vias 0 -> 3
- net Row6: track 227.5 -> 0.00 mm, vias 6 -> 0
- net Col10: track 0.00 -> 195.6 mm
- net Row9: track 194.0 -> 0.00 mm, vias 2 -> 0
- net Col6: track 448.5 -> 267.2 mm, vias 5 -> 0
- net Row8: track 178.0 -> 0.00 mm, vias 4 -> 0
- net Row7: track 177.9 -> 0.00 mm, vias 4 -> 0
- net Col11: track 0.00 -> 172.4 mm
- net Col12: track 0.00 -> 159.3 mm, vias 0 -> 3
- net Col13: track 0.00 -> 155.7 mm, vias 0 -> 3
- net Col3: track 433.5 -> 286.3 mm, vias 2 -> 0
- net Col17: track 0.00 -> 133.4 mm, vias 0 -> 2
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Other:
- net class Default: clearance 0.2 -> 0.158
- net class Power: clearance 0.2 -> 0.158
- rule trace_clearance: 0.2 -> 0.158
- rule trace_min: 0.2 -> 0.158
- board text added: "B15"
- board text added: "Rev. 6"
- board text removed: "E6"
- board text removed: "Rev. 5.1"

Commit message: Rerouted, added render
Parts:
- added svg2mod: G***, Artwork:CableCarLogo, B.Cu at (275.5, 196.3)
- added svg2mod: G***, Artwork:CableCarLogo, F.Cu at (275.5, 196.3)
- moved R92 12.6 mm to (392.0, 122.3)
- moved D64 12.5 mm to (270.6, 154.4)
- moved D70 6.80 mm to (308.7, 116.3)
- moved C6 4.98 mm to (325.3, 163.4)
- moved U1 3.70 mm to (315.8, 161.6)
- moved D66 3.64 mm to (306.3, 144.9)
- moved C5 2.85 mm to (321.5, 170.1)
- moved D90 2.84 mm to (378.9, 183.0)
- moved R28 2.77 mm to (202.7, 109.2)
- moved D7 2.39 mm to (42.0, 116.3)
- moved U2 2.22 mm to (215.8, 116.3)
- moved D45 1.82 mm to (211.0, 192.5)
- moved D20 1.77 mm to (130.1, 192.5)
- moved C4 1.63 mm to (324.1, 159.2), turned to 270 degrees
- moved D92 1.59 mm to (208.7, 192.5)
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Connections:
- U1 pad 10: Net-(U1-Pad10) -> Col18
- U1 pad 2: Col16 -> Col17
- U1 pad 3: Col17 -> Col16
Routing:
- net Col18: track 83.8 -> 165.3 mm, vias 2 -> 0
- net Net-(U1-Pad10): track 80.4 -> 0.00 mm, vias 2 -> 0
- net Col8: track 284.1 -> 206.7 mm, vias 0 -> 2
- net LEDGND: track 1799.5 -> 1858.4 mm, vias 17 -> 20
- net Row1: track 398.5 -> 437.8 mm
- net +5V: track 2240.7 -> 2201.6 mm, vias 3 -> 5
- net Col6: track 267.2 -> 293.7 mm, vias 0 -> 2
- net Col2: track 346.4 -> 372.2 mm, vias 0 -> 2
- net Row0: track 441.7 -> 466.2 mm, vias 2 -> 6
- net Row3: track 387.0 -> 405.9 mm, vias 4 -> 6
- net Col7: track 254.1 -> 272.1 mm, vias 0 -> 2
- net Col12: track 159.3 -> 143.8 mm, vias 3 -> 1
- net +3V3: track 242.4 -> 227.8 mm, vias 3 -> 7
- net NRST: track 50.0 -> 62.2 mm
- net Col13: track 155.7 -> 166.4 mm, vias 3 -> 1
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