File: cypher.kicad_pcb (KiCad board)
At the start: 2 copper layers, 370.1 x 106 mm, 309 parts, among them J3 Breakout, Q1 BC850, Q2 MMBT3904, SW1 SW_Push, U1 STM32F072CBTx, U2 PRTR5V0U2X, U3 LD3985G33R_TSOT23

Commit message: updated rev6
Parts:
- D10, D11, D12, D13, D14, D15, D16, D17, D18, D19, D20, D21, D22, D23, D24, D25, D26, D27, D28, D29, D30, D31, D32, D33, D34, D35, D36, D37, D38, D39, D4, D40, D41, D42, D43, D44, D45, D46, D47, D48, D49, D5, D50, D51, D52, D53, D54, D55, D56, D57, D58, D59, D6, D60, D61, D62, D63, D64, D65, D66, D67, D68, D69, D7, D70, D71, D72, D73, D74, D75, D76, D77, D78, D79, D8, D80, D81, D82, D83, D84, D85, D86, D87, D88, D89, D9, D90, D92: footprint Diode_SMD:D_0603_1608Metric -> Diode_SMD:D_SOD-123
- D91: value D -> 1N4148; footprint Diode_SMD:D_0603_1608Metric -> Diode_SMD:D_SOD-123
- moved D15 2.38 mm to (82.4, 116.3)
- moved D29 1.19 mm to (138.4, 116.3)
- moved D24 1.19 mm to (119.4, 116.3)
- moved D21 1.19 mm to (100.3, 116.3)
- moved D11 1.19 mm to (62.2, 116.3)
- moved D7 1.19 mm to (43.2, 116.3)
- moved D26 1.19 mm to (133.6, 154.4)
- moved D32 1.19 mm to (169.4, 192.5)
- moved D34 1.19 mm to (157.5, 116.3)
- moved D37 1.19 mm to (181.3, 173.5)
- moved D43 1.19 mm to (205.1, 135.4)
- moved D47 1.19 mm to (228.9, 154.4)
- moved D56 1.19 mm to (252.7, 116.3)
- moved D10 1.19 mm to (67.0, 173.5)
- moved D12 1.19 mm to (71.7, 135.4)
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Routing:
- net Row1: track 437.8 -> 387.8 mm
- net Row0: track 466.2 -> 439.4 mm
- net Row3: track 405.9 -> 431.4 mm
- net Row2: track 395.1 -> 376.7 mm
- net Row4: track 421.7 -> 404.6 mm
- net Net-(D91-Pad2): track 137.3 -> 141.7 mm
- net Net-(D39-Pad2): track 6.39 -> 9.31 mm
- net Net-(D9-Pad2): track 36.9 -> 39.5 mm
- net Net-(D15-Pad2): track 6.39 -> 8.72 mm
- net Net-(D24-Pad2): track 6.39 -> 8.70 mm
- net Net-(D92-Pad2): track 18.4 -> 16.7 mm
- net Col18: track 165.3 -> 166.7 mm
- net Col13: track 166.4 -> 165.1 mm
- net Col7: track 272.1 -> 270.8 mm
- net Net-(D67-Pad2): track 6.60 -> 7.79 mm
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
Commit message: updated rev6
Parts:
- added C10: 100nf, Capacitor_SMD:C_0603_1608Metric, F.Cu at (320.1, 119.5)
- added C8: 100nf, Capacitor_SMD:C_0603_1608Metric, F.Cu at (320.1, 113.2)
- added C9: 100nf, Capacitor_SMD:C_0603_1608Metric, F.Cu at (320.1, 116.5)
Connections:
- U1 pad 25: Col5 -> Net-(U1-Pad25)
- U1 pad 26: Col4 -> Net-(U1-Pad26)
- U1 pad 27: Col3 -> Net-(U1-Pad27)
- U1 pad 40: Net-(U1-Pad40) -> Col3
- U1 pad 41: Net-(U1-Pad41) -> Col4
- U1 pad 42: Net-(U1-Pad42) -> Col5
Routing:
- net Col5: track 248.9 -> 265.8 mm, vias 2 -> 4
- net Col4: track 295.7 -> 312.6 mm, vias 2 -> 4
- net Col3: track 291.2 -> 305.5 mm, vias 2 -> 4
- net +5V: track 2201.6 -> 2212.8 mm
- net LED_OUT: track 52.1 -> 57.3 mm
- net Net-(D1-Pad4): track 2.87 -> 8.07 mm
- net Net-(D2-Pad4): track 2.77 -> 7.51 mm
- net B15: track 28.8 -> 30.9 mm
- net Row1: track 387.8 -> 388.3 mm
- net GND: vias 22 -> 24
