File: cypher.kicad_pcb (KiCad board)
At the start: 2 copper layers, 370.1 x 107.1 mm, 298 parts, among them J1 USB_B_Mini, J2 AVR-ISP-6, Q1 Q_NPN_BCE, SW1 SW_Push, U1 ATmega32U4-AU, Y1 16Mhz

Commit message: Update files to rev. 2
correction of error in the crystal wiring

adjusted all the diode footprints to be easier to read

moved D70 to be vertical and placed more in line with the rest of the diodes

bumped silkscreen to rev. 2
Parts:
- D10, D11, D12, D13, D14, D15, D16, D17, D18, D19, D21, D22, D23, D24, D25, D26, D27, D28, D29, D30, D31, D32, D33, D34, D35, D36, D37, D38, D39, D4, D40, D41, D42, D43, D44, D45, D46, D47, D48, D49, D5, D50, D51, D52, D53, D54, D55, D56, D57, D58, D59, D6, D60, D61, D62, D63, D64, D65, D66, D67, D68, D69, D7, D70, D71, D72, D73, D74, D75, D76, D77, D78, D79, D8, D80, D81, D82, D83, D84, D85, D86, D87, D88, D89, D9, D90: value D_Small -> 1N4148
- J2: moved to B.Cu
- R10, R11, R12, R13, R14, R15, R16, R17, R18, R19, R20, R21, R22, R23, R24, R25, R26, R27, R29, R30, R31, R32, R33, R34, R35, R36, R37, R38, R39, R40, R41, R42, R43, R44, R45, R46, R47, R48, R49, R50, R51, R52, R53, R54, R55, R56, R57, R58, R59, R6, R60, R61, R62, R63, R64, R65, R66, R67, R68, R69, R7, R70, R71, R72, R73, R74, R75, R76, R77, R78, R79, R8, R80, R81, R82, R83, R84, R85, R86, R87, R88, R89, R9, R90, R91, R92, R93, R94, R95: value 1K -> 470
- moved D70 16.3 mm to (310.7, 100.0), turned to 90 degrees
- moved C2 0.85 mm to (180.3, 191.9)
- moved C3 0.67 mm to (191.2, 191.8)
- turned J2 to 180 degrees
- turned Y1 to 0 degrees
Connections:
- J1 pad 4: Net-(J1-Pad4) -> (no net)
- U1 pad 36: Net-(U1-Pad36) -> (no net)
- U1 pad 42: Net-(U1-Pad42) -> (no net)
- Y1 pad 1: GND -> XTAL1
- Y1 pad 2: XTAL1 -> GND
- Y1 pad 3: GND -> XTAL2
- Y1 pad 4: XTAL2 -> GND
Routing:
- net GND: track 227.6 -> 248.5 mm, vias 58 -> 59
- net Net-(D70-Pad2): track 12.2 -> 5.36 mm
- net Row1: track 284.0 -> 287.8 mm
- net RESET: track 94.1 -> 97.0 mm
- net MISO: track 218.8 -> 221.4 mm
- net XTAL1: track 11.5 -> 8.91 mm
- net +5V: track 2058.7 -> 2056.5 mm
- net XTAL2: track 11.4 -> 13.5 mm
- net MOSI: track 256.3 -> 254.3 mm
- net Row5: track 284.9 -> 285.8 mm
Other:
- board text added: "Rev. 2"
- board text removed: "Rev. 1"

Commit message: updated to rev.3
Parts:
- added svg2mod: G***, Artwork:AFbw, B.Cu at (106.4, 182.9)
- C8: footprint Diode_SMD:D_0805_2012Metric_Pad1.15x1.40mm_HandSolder -> Capacitor_SMD:C_0805_2012Metric_Pad1.15x1.40mm_HandSolder
- moved R92 12.4 mm to (381.8, 112.9)
- moved D66 10.4 mm to (309.6, 138.9)
- moved D85 4.44 mm to (377.8, 164.3)
- moved D90 4.44 mm to (381.0, 170.7)
- moved D81 4.34 mm to (377.8, 126.2)
- moved D86 4.02 mm to (377.8, 178.6)
- moved R93 3.87 mm to (381.8, 131.8)
- moved R71 3.72 mm to (307.2, 131.9)
- moved D34 2.65 mm to (158.8, 107.0)
- moved D22 2.34 mm to (111.1, 126.2)
- moved D6 2.32 mm to (49.2, 183.4)
- moved D68 2.29 mm to (315.9, 188.1)
- moved D88 2.23 mm to (377.8, 131.8)
- moved D74 2.20 mm to (339.7, 164.3)
- moved D48 1.52 mm to (200.8, 107.0)
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Routing:
- net GND: track 248.5 -> 454.0 mm, vias 59 -> 14
- net Col0: track 424.9 -> 571.7 mm, vias 2 -> 1
- net Col1: track 428.4 -> 557.1 mm, vias 2 -> 3
- net LEDGND: track 1786.7 -> 1900.6 mm, vias 27 -> 4
- net +5V: track 2056.5 -> 2136.8 mm, vias 13 -> 10
- net Scrl: track 185.2 -> 240.3 mm, vias 5 -> 1
- net Row9: track 221.3 -> 275.5 mm, vias 4 -> 2
- net Num: track 190.3 -> 243.5 mm, vias 5 -> 1
- net Col3: track 458.2 -> 509.0 mm, vias 2 -> 3
- net Net-(R5-Pad2): track 185.8 -> 226.8 mm, vias 6 -> 2
- net Caps: track 207.7 -> 246.7 mm, vias 5 -> 1
- net Col5: track 392.6 -> 427.9 mm, vias 4 -> 3
- net Row0: track 257.7 -> 291.8 mm, vias 4 -> 2
- net Col8: track 404.7 -> 372.3 mm, vias 7 -> 4
- net Row4: track 170.7 -> 193.8 mm
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Other:
- net class Default: trace_width 0.25 -> 0.254
- net class Power added: clearance 0.2, trace_width 0.381, via_dia 0.8, via_drill 0.4
- board text added: "Rev. 3"
- board text removed: "Rev. 2"

Commit message: update to rev5
Parts:
- removed F1: 500ma, Fuse:Fuse_0805_2012Metric_Pad1.15x1.40mm_HandSolder
- removed J1: USB_B_Mini, Connector_USB:U-M-M5DD-W-1
- removed the svg2mod at (106.4, 182.9)
- added D20: 1N4148, Diode_SMD:D_0603_1608Metric, B.Cu at (131.7, 193.3)
- added D92: 1N4148, Diode_SMD:D_0603_1608Metric, B.Cu at (207.1, 192.5)
- added Fe: 500ma, Fuse:Fuse_0805_2012Metric, B.Cu at (220.0, 107.5)
- added J3: Breakout, Connector_PinHeader_2.54mm:PinHeader_1x03_P2.54mm_Vertical, F.Cu at (337.7, 186.1)
- added MX101: Split_left, 19mmMX:MXOnly-2.75U-FLIPPED-ReversedStabilizers, F.Cu at (122.9, 192.5)
- added MX102: Split_left, MX_Only:MXOnly-2.25U-ReversedStabilizers, F.Cu at (118.2, 192.5)
- added MX103: Split_center, MX_Only:MXOnly-1.25U, F.Cu at (151.5, 192.5)
- added MX104: Split_center, 19mmMX:MXOnly-1.25U-FLIPPED, F.Cu at (161.0, 192.5)
- added MX105: Split_right, MX_Only:MXOnly-2.25U-ReversedStabilizers, F.Cu at (194.4, 192.5)
- added MX106: Split_right, 19mmMX:MXOnly-2.75U-FLIPPED-ReversedStabilizers, F.Cu at (189.6, 192.5)
- added R28: 5.1K, Resistor_SMD:R_0603_1608Metric, B.Cu at (205.4, 109.9)
- added R96: 5.1K, Resistor_SMD:R_0603_1608Metric, B.Cu at (220.0, 109.3)
- added R97: 470, Resistor_SMD:R_0603_1608Metric, B.Cu at (126.9, 198.9)
- added R99: 470, Resistor_SMD:R_0603_1608Metric, B.Cu at (185.6, 198.1)
- added U2: PRTR5V0U2X, PRTR5V0U2X:SOT143B, B.Cu at (216.9, 114.2)
- added USB1: HRO-TYPE-C-31-M-12, Type-C:HRO-TYPE-C-31-M-12, B.Cu at (210.7, 100.4)
- added svg2mod: G***, Artwork:CableCarLogo, B.Cu at (285.5, 183.9)
- C1: value 4.7uf -> 4.7uF; footprint Capacitor_SMD:C_0805_2012Metric_Pad1.15x1.40mm_HandSolder -> Capacitor_SMD:C_0603_1608Metric
- C2, C3: value 22p -> 22pF; footprint Capacitor_SMD:C_0805_2012Metric_Pad1.15x1.40mm_HandSolder -> Capacitor_SMD:C_0603_1608Metric
- C4, C5, C6, C7: value 0.1uf -> 100nF; footprint Capacitor_SMD:C_0805_2012Metric_Pad1.15x1.40mm_HandSolder -> Capacitor_SMD:C_0603_1608Metric
- C8: footprint Capacitor_SMD:C_0805_2012Metric_Pad1.15x1.40mm_HandSolder -> Capacitor_SMD:C_0603_1608Metric
- D10, D11, D12, D13, D14, D15, D16, D17, D18, D19, D21, D22, D23, D24, D25, D26, D27, D28, D29, D30, D31, D32, D33, D34, D35, D36, D37, D38, D39, D4, D40, D41, D42, D43, D44, D45, D46, D47, D48, D49, D5, D50, D51, D52, D53, D54, D55, D56, D57, D58, D59, D6, D60, D61, D62, D63, D64, D65, D66, D67, D68, D69, D7, D70, D71, D72, D73, D74, D75, D76, D77, D78, D79, D8, D80, D81, D82, D83, D84, D85, D86, D87, D88, D89, D9, D90: footprint Diode_SMD:D_0805_2012Metric_Pad1.15x1.40mm_HandSolder -> Diode_SMD:D_0603_1608Metric
- J2: footprint Molex-0548190589:Reset_Pretty-Mask -> Connector_PinHeader_2.54mm:PinHeader_2x03_P2.54mm_Vertical
- MX1, MX75: footprint MX_Alps_Hybrid:MXOnly-2.25U -> MX_Only:MXOnly-2.25U
- MX10, MX11, MX12, MX13, MX14, MX16, MX17, MX18, MX19, MX21, MX22, MX23, MX24, MX26, MX27, MX28, MX29, MX30, MX31, MX32, MX33, MX36, MX37, MX38, MX39, MX4, MX41, MX42, MX43, MX44, MX45, MX46, MX47, MX48, MX49, MX50, MX51, MX52, MX55, MX56, MX57, MX58, MX59, MX61, MX62, MX63, MX64, MX66, MX67, MX68, MX70, MX71, MX76, MX77, MX78, MX79, MX80, MX81, MX82, MX83, MX84, MX85, MX86, MX87, MX88, MX89, MX90, MX91, MX92, MX93, MX94, MX95, MX96, MX97, MX99: footprint MX_Alps_Hybrid:MXOnly-1U -> MX_Only:MXOnly-1U
- MX100, MX98: footprint MX_Alps_Hybrid:MXOnly-2U-ReversedStabilizers -> MX_Only:MXOnly-2U-ReversedStabilizers
- MX15, MX5, MX54, MX60, MX74: footprint MX_Alps_Hybrid:MXOnly-1.5U -> MX_Only:MXOnly-1.5U
- MX2: footprint MX_Alps_Hybrid:MXOnly-1.5U-FLIPPED -> MX_Only:MXOnly-1.5U-FLIPPED
- MX20, MX3, MX53, MX7, MX8: footprint MX_Alps_Hybrid:MXOnly-1.25U -> MX_Only:MXOnly-1.25U
- MX25, MX65: footprint MX_Alps_Hybrid:MXOnly-1.25U-FLIPPED -> MX_Only:MXOnly-1.25U-FLIPPED
- MX34: footprint MX_Alps_Hybrid:MXOnly-6.25U-FLIPPED-ReversedStabilizers -> MX_Only:MXOnly-6.25U-FLIPPED-ReversedStabilizers
- MX35: footprint MX_Alps_Hybrid:MXOnly-7U-ReversedStabilizers -> 19mmMX:MXOnly-7U-FLIPPED-ReversedStabilizers
- MX40: footprint MX_Alps_Hybrid:MXOnly-6U-ReversedStabilizers -> MX_Only:MXOnly-6U-ReversedStabilizers
- MX6: footprint MX_Alps_Hybrid:MXOnly-1.75U-FLIPPED -> MX_Only:MXOnly-1.75U-FLIPPED
- MX69: footprint MX_Alps_Hybrid:MXOnly-1.75U -> MX_Only:MXOnly-1.75U
- MX72: footprint MX_Alps_Hybrid:MXOnly-ISO-ROTATED-ReversedStabilizers -> MX_Only:MXOnly-ISO-ReversedStabilizers
- MX73: footprint MX_Alps_Hybrid:MXOnly-2U -> MX_Only:MXOnly-2U
- MX9: footprint MX_Alps_Hybrid:MXOnly-1.25U-FLIPPED -> MX_Only:MXOnly-1U-FLIPPED
- Q1: footprint Package_TO_SOT_SMD:SOT-223-3_TabPin2 -> Package_TO_SOT_SMD:SOT-23
- R1, R10, R11, R12, R13, R14, R15, R16, R17, R18, R19, R2, R20, R21, R22, R23, R24, R25, R26, R27, R29, R3, R30, R31, R32, R33, R34, R35, R36, R37, R38, R39, R4, R40, R41, R42, R43, R44, R45, R46, R47, R48, R49, R5, R50, R51, R52, R53, R54, R55, R56, R57, R58, R59, R6, R60, R61, R62, R63, R64, R65, R66, R67, R68, R69, R7, R70, R71, R72, R73, R74, R75, R76, R77, R78, R79, R8, R80, R81, R82, R83, R84, R85, R86, R87, R88, R89, R9, R90, R91, R92, R93, R94, R95: footprint Resistor_SMD:R_0805_2012Metric_Pad1.15x1.40mm_HandSolder -> Resistor_SMD:R_0603_1608Metric
- SW1: value SW_Push -> RESET; footprint Button_Switch_SMD:SW_SPST_TL3342 -> Connector_PinHeader_2.54mm:PinHeader_2x01_P2.54mm_Vertical
- U1: value ATmega32U4-AU -> ATmega32U4-MU; footprint Package_QFP:TQFP-44_10x10mm_P0.8mm -> Package_DFN_QFN:QFN-44-1EP_7x7mm_P0.5mm_EP5.2x5.2mm
- Y1: footprint Crystal:Crystal_SMD_3225-4Pin_3.2x2.5mm_HandSoldering -> Crystal:Crystal_SMD_2520-4Pin_2.5x2.0mm
- moved R3 179.4 mm to (313.3, 152.9)
- moved C4 145.6 mm to (315.6, 152.9), turned to 270 degrees
- moved C2 145.5 mm to (321.6, 157.0), turned to 135 degrees
- moved R4 142.1 mm to (315.7, 173.4), turned to 45 degrees
- moved Y1 137.4 mm to (318.8, 157.6), turned to 135 degrees
- moved C3 133.5 mm to (319.4, 154.8), turned to 315 degrees
- moved C6 130.2 mm to (312.7, 172.6), turned to 315 degrees
- moved U1 129.4 mm to (313.6, 164.0), turned to 315 degrees
- moved C5 123.7 mm to (321.5, 167.5), turned to 225 degrees
- moved C8 116.2 mm to (311.8, 152.9)
- moved C7 113.7 mm to (306.3, 167.0), turned to 135 degrees
- moved C1 112.6 mm to (306.7, 161.3), turned to 45 degrees
- moved J2 81.4 mm to (295.2, 181.2)
- moved SW1 27.0 mm to (104.4, 192.5), turned to 180 degrees
- moved Q1 21.5 mm to (314.7, 127.1), turned to 180 degrees
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Connections:
- D10 pad 1: MISO -> Row3
- D13 pad 1: MOSI -> Row2
- D17 pad 1: MOSI -> Row2
- D18 pad 1: MISO -> Row3
- D19 pad 1: MOSI -> Row2
- D23 pad 1: MISO -> Row3
- D26 pad 1: MOSI -> Row2
- D27 pad 1: MISO -> Row3
- D28 pad 1: MISO -> Row3
- D31 pad 1: MOSI -> Row2
- D33 pad 1: MISO -> Row3
- D36 pad 1: MOSI -> Row2
- D37 pad 1: MISO -> Row3
- D4 pad 1: MOSI -> Row2
- D40 pad 1: MOSI -> Row2
- D41 pad 1: MISO -> Row3
- D44 pad 1: MOSI -> Row2
- D46 pad 1: MISO -> Row3
- D47 pad 1: MOSI -> Row2
- D5 pad 1: MISO -> Row3
- J2 pad 1: MISO -> Col6
- J2 pad 3: Row1 -> Col8
- J2 pad 4: MOSI -> Col7
- R1 pad 1: D+ -> D-
- R2 pad 1: D- -> D+
- U1 pad 1: Col8 -> E6
- U1 pad 10: MOSI -> Col7
- U1 pad 11: MISO -> Col6
- U1 pad 12: Row7 -> Col5
- U1 pad 18: Col0 -> Net-(R5-Pad2)
- U1 pad 19: Col1 -> Row5
- U1 pad 20: Col2 -> Scrl
- U1 pad 21: Col3 -> Num
- U1 pad 22: Col5 -> Caps
- U1 pad 25: Col4 -> Row7
- U1 pad 26: Col6 -> Col0
- U1 pad 27: Col7 -> Col1
- U1 pad 28: Row4 -> Col2
- U1 pad 29: Net-(R5-Pad2) -> Col3
- U1 pad 30: Row6 -> Col4
- U1 pad 36: (no net) -> Row4
- U1 pad 37: Row5 -> Row3
- U1 pad 38: Scrl -> Row2
- U1 pad 39: Num -> Row6
- U1 pad 40: Caps -> Row1
- U1 pad 9: Row1 -> Col8
Routing:
- net Row2: track 0.00 -> 312.8 mm, vias 0 -> 6
- net GND: track 454.0 -> 146.0 mm, vias 14 -> 29
- net Row3: track 0.00 -> 280.1 mm, vias 0 -> 2
- net MOSI: track 275.2 -> 0.00 mm, vias 4 -> 0
- net MISO: track 231.0 -> 0.00 mm, vias 4 -> 0
- net +5V: track 2136.8 -> 2341.1 mm, vias 10 -> 11
- net RESET: track 119.6 -> 312.7 mm, vias 2 -> 1
- net Scrl: track 240.3 -> 51.5 mm, vias 1 -> 0
- net Net-(R5-Pad2): track 226.8 -> 40.6 mm, vias 2 -> 0
- net Num: track 243.5 -> 60.1 mm, vias 1 -> 0
- net Caps: track 246.7 -> 63.8 mm, vias 1 -> 0
- net Col7: track 383.4 -> 496.9 mm, vias 3 -> 8
- net Row4: track 193.8 -> 299.4 mm, vias 3 -> 4
- net LEDGND: track 1900.6 -> 1798.0 mm, vias 4 -> 19
- net Col1: track 557.1 -> 465.5 mm, vias 3 -> 4
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Other:
- board size 370.1 x 107.1 mm -> 370.1 x 106 mm
- board text added: "+5V"
- board text added: "E6"
- board text added: "GND"
- board text added: "Rev. 5"
- board text removed: "Rev. 3"

Commit message: updated to rev 5.1
Parts:
- Q1: value Q_NPN_BCE -> MMBT3904
- SW1: value RESET -> SW_Push
- moved Q1 0.38 mm to (314.4, 127.1)
- renumbered Fe to F1
Connections:
- Q1 pad 2: LEDGND -> GND
- Q1 pad 3: GND -> LEDGND
- U1 pad 42: (no net) -> Net-(U1-Pad42)
- USB1 pad 3: (no net) -> Net-(USB1-Pad3)
- USB1 pad 9: (no net) -> Net-(USB1-Pad9)
Routing:
- net LEDGND: track 1798.0 -> 1801.0 mm
- net GND: track 146.0 -> 147.0 mm
Other:
- board text added: "Rev. 5.1"
- board text removed: "Rev. 5"

Commit message: Cleanup and commit for rev6
Parts:
- removed R6, R7, R8: 470, Resistor_SMD:R_0603_1608Metric
- added C10: 100nf, Capacitor_SMD:C_0603_1608Metric, F.Cu at (319.6, 116.5)
- added C11: 100nf, Capacitor_SMD:C_0603_1608Metric, F.Cu at (319.6, 119.7)
- added C9: 100nf, Capacitor_SMD:C_0603_1608Metric, F.Cu at (319.6, 113.4)
- D1: value CAPS -> WS2812B; footprint LED_THT:LED_D1.8mm_W3.3mm_H2.4mm -> CrumpPrints:WS2812-2020
- D2: value Num -> WS2812B; footprint LED_THT:LED_D1.8mm_W3.3mm_H2.4mm -> CrumpPrints:WS2812-2020
- D3: value Scroll -> WS2812B; footprint LED_THT:LED_D1.8mm_W3.3mm_H2.4mm -> CrumpPrints:WS2812-2020
- moved D1 1.31 mm to (315.8, 113.2)
- moved D3 1.30 mm to (315.8, 119.5)
- moved D2 1.29 mm to (315.8, 116.3)
Connections:
- D1 pad 1: Net-(D1-Pad1) -> +5V
- D1 pad 2: Caps -> D5
- D2 pad 1: Net-(D2-Pad1) -> +5V
- D2 pad 2: Num -> Net-(D1-Pad4)
- D3 pad 1: Net-(D3-Pad1) -> +5V
- D3 pad 2: Scrl -> Net-(D2-Pad4)
Routing:
- net Num: track 60.1 -> 0.00 mm
- net Scrl: track 51.5 -> 0.00 mm
- net +5V: track 2341.1 -> 2368.9 mm, vias 11 -> 12
- net Caps: track 63.8 -> 55.9 mm, vias 0 -> 1
- net Net-(D2-Pad4): track 0.00 -> 7.60 mm
- net Net-(D1-Pad4): track 0.00 -> 7.36 mm
- net Net-(D2-Pad1): track 2.79 -> 0.00 mm
- net Net-(D3-Pad1): track 2.79 -> 0.00 mm
- net Net-(D1-Pad1): track 2.74 -> 0.00 mm
- net GND: vias 29 -> 32
Other:
- rule pad_to_mask_clearance: 0.2 -> 0
- board text added: "Rev. 6"
- board text removed: "Rev. 5.1"
