File: cypher.sch (KiCad schematic (older format))
At the start: 26 parts, among them J1 USB_B_Mini, J2 AVR-ISP-6, Q1 Q_NPN_BCE, SW1 SW_Push, U1 ATmega32U4-AU, Y1 16Mhz

Commit message: Update files to rev. 2
correction of error in the crystal wiring

adjusted all the diode footprints to be easier to read

moved D70 to be vertical and placed more in line with the rest of the diodes

bumped silkscreen to rev. 2
Parts:
- R6, R7, R8: value 1K -> 470
Changed lines of the file:
@@
 $EndComp
 Wire Wire Line
-	1425 2725 1425 2700
+	1425 2775 1425 2700
 $Comp
 L Device:Crystal_GND24 Y1
@@
 F 3 "~" H 1425 2925 50  0001 C CNN
 	1    1425 2925
-	1    0    0    -1
-$EndComp
-Wire Wire Line
-	1425 3150 1425 3125
+	0    1    1    0
+$EndComp
+Wire Wire Line
+	1425 3150 1425 3075
 Text GLabel 1770 2700 2    50   Input ~ 0
 XTAL1
@@
 	1425 2700 1770 2700
 Wire Wire Line
-	1575 2925 1600 2925
-Wire Wire Line
-	1600 2925 1600 3425
-Wire Wire Line
-	1600 3425 1250 3425
-Wire Wire Line
-	1250 3425 1250 2925
-Wire Wire Line
-	1250 2925 1275 2925
-Wire Wire Line
-	1250 3425 625  3425
+	1650 3425 1200 3425
+Wire Wire Line
+	1200 3425 1200 2925
+Wire Wire Line
+	1200 2925 1225 2925
+Wire Wire Line
+	1200 3425 625  3425
 Wire Wire Line
 	625  3425 625  3150
 Wire Wire Line
 	625  2700 800  2700
-Connection ~ 1250 3425
+Connection ~ 1200 3425
 Wire Wire Line
 	800  3150 625  3150
@@
 L power:GND #PWR0101
 U 1 1 5C12C2C7
-P 1250 3425
-F 0 "#PWR0101" H 1250 3175 50  0001 C CNN
-F 1 "GND" H 1255 3252 50  0000 C CNN
-F 2 "" H 1250 3425 50  0001 C CNN
-F 3 "" H 1250 3425 50  0001 C CNN
-	1    1250 3425
+P 1200 3425
+F 0 "#PWR0101" H 1200 3175 50  0001 C CNN
+F 1 "GND" H 1205 3252 50  0000 C CNN
+F 2 "" H 1200 3425 50  0001 C CNN
+F 3 "" H 1200 3425 50  0001 C CNN
+	1    1200 3425
 	1    0    0    -1
 $EndComp
@@
 P 5350 1100
 F 0 "R6" V 5154 1100 50  0000 C CNN
-F 1 "1K" V 5245 1100 50  0000 C CNN
+F 1 "470" V 5245 1100 50  0000 C CNN
 F 2 "Resistor_SMD:R_0805_2012Metric_Pad1.15x1.40mm_HandSolder" H 5350 1100 50  0001 C CNN
 F 3 "~" H 5350 1100 50  0001 C CNN
@@
 P 5350 1375
 F 0 "R7" V 5154 1375 50  0000 C CNN
-F 1 "1K" V 5245 1375 50  0000 C CNN
+F 1 "470" V 5245 1375 50  0000 C CNN
 F 2 "Resistor_SMD:R_0805_2012Metric_Pad1.15x1.40mm_HandSolder" H 5350 1375 50  0001 C CNN
 F 3 "~" H 5350 1375 50  0001 C CNN
@@
 P 5350 1650
 F 0 "R8" V 5154 1650 50  0000 C CNN
-F 1 "1K" V 5245 1650 50  0000 C CNN
+F 1 "470" V 5245 1650 50  0000 C CNN
 F 2 "Resistor_SMD:R_0805_2012Metric_Pad1.15x1.40mm_HandSolder" H 5350 1650 50  0001 C CNN
 F 3 "~" H 5350 1650 50  0001 C CNN
@@
 Wire Wire Line
 	3100 2275 3425 2275
+Wire Wire Line
+	1625 2925 1650 2925
+Wire Wire Line
+	1650 2925 1650 3425
 $EndSCHEMATC

Commit message: update to rev5
Parts:
- removed J1: USB_B_Mini, Connector_USB:U-M-M5DD-W-1, symbol Connector:USB_B_Mini
- removed U1: ATmega32U4-AU, Package_QFP:TQFP-44_10x10mm_P0.8mm, symbol MCU_Microchip_ATmega:ATmega32U4-AU
- added J3: Breakout, Connector_PinHeader_2.54mm:PinHeader_1x03_P2.54mm_Vertical, symbol Connector:Conn_01x03_Male
- added R28, R96: 5.1K, Resistor_SMD:R_0603_1608Metric, symbol Device:R_Small
- added U1: ATmega32U4-MU, Package_DFN_QFN:QFN-44-1EP_7x7mm_P0.5mm_EP5.2x5.2mm, symbol MCU_Microchip_ATmega:ATmega32U4-MU
- added U2: PRTR5V0U2X, PRTR5V0U2X:SOT143B, symbol ai03-locallib:PRTR5V0U2X
- added USB1: HRO-TYPE-C-31-M-12, Type-C:HRO-TYPE-C-31-M-12, symbol Type-C:HRO-TYPE-C-31-M-12
- C1: value 4.7uf -> 4.7uF; footprint Capacitor_SMD:C_0805_2012Metric_Pad1.15x1.40mm_HandSolder -> Capacitor_SMD:C_0603_1608Metric
- C2, C3: value 22p -> 22pF; footprint Capacitor_SMD:C_0805_2012Metric_Pad1.15x1.40mm_HandSolder -> Capacitor_SMD:C_0603_1608Metric
- C4, C5, C6, C7: value 0.1uf -> 100nF; footprint Capacitor_SMD:C_0805_2012Metric_Pad1.15x1.40mm_HandSolder -> Capacitor_SMD:C_0603_1608Metric
- C8: footprint Diode_SMD:D_0805_2012Metric_Pad1.15x1.40mm_HandSolder -> Capacitor_SMD:C_0603_1608Metric
- F1: footprint Fuse:Fuse_0805_2012Metric_Pad1.15x1.40mm_HandSolder -> Fuse:Fuse_0805_2012Metric
- J2: footprint Molex-0548190589:Reset_Pretty-Mask -> Connector_PinHeader_2.54mm:PinHeader_2x03_P2.54mm_Vertical
- Q1: footprint Package_TO_SOT_SMD:SOT-223-3_TabPin2 -> Package_TO_SOT_SMD:SOT-23
- R1, R2, R3, R4, R5, R6, R7, R8: footprint Resistor_SMD:R_0805_2012Metric_Pad1.15x1.40mm_HandSolder -> Resistor_SMD:R_0603_1608Metric
- SW1: footprint Button_Switch_SMD:SW_SPST_TL3342 -> Connector_PinHeader_2.54mm:PinHeader_2x01_P2.54mm_Vertical
- Y1: footprint Crystal:Crystal_SMD_3225-4Pin_3.2x2.5mm_HandSoldering -> Crystal:Crystal_SMD_2520-4Pin_2.5x2.0mm
Connections:
- net labels added: E6
- wire segments 112 -> 147
Other:
- moved on the sheet: C1, C2, C3, C4, C5, C6, C7, C8, D1, D2, D3, F1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

Commit message: updated to rev 5.1
Parts:
- removed Q1: Q_NPN_BCE, Package_TO_SOT_SMD:SOT-23, symbol Device:Q_NPN_BCE
- added Q1: MMBT3904, Package_TO_SOT_SMD:SOT-23, symbol transistors:MMBT3904
Connections:
- net GND: now also Q1.2 (E)
- net LEDGND: now also Q1.3 (C)
- net at R5.1: now also Q1.1 (B)
Other:
- moved on the sheet: D1, D2, D3, R6, R7, R8
Changed lines of the file:
@@
 EESchema Schematic File Version 4
-LIBS:cypher-cache
-EELAYER 29 0
+EELAYER 30 0
 EELAYER END
 $Descr A4 11693 8268
@@
 	3665 6495 3940 6495
 $Comp
-L Device:Q_NPN_BCE Q1
-U 1 1 5C16E6B4
-P 5390 4995
-F 0 "Q1" H 5581 5041 50  0000 L CNN
-F 1 "Q_NPN_BCE" H 5581 4950 50  0000 L CNN
-F 2 "Package_TO_SOT_SMD:SOT-23" H 5590 5095 50  0001 C CNN
-F 3 "~" H 5390 4995 50  0001 C CNN
-	1    5390 4995
-	1    0    0    -1
-$EndComp
-$Comp
 L power:VCC #PWR0112
 U 1 1 5C16E7F6
@@
 	4790 4995 5190 4995
 $Comp
-L Device:R_Small R6
-U 1 1 5C1827C5
-P 7130 1660
-F 0 "R6" V 6934 1660 50  0000 C CNN
-F 1 "470" V 7025 1660 50  0000 C CNN
-F 2 "Resistor_SMD:R_0603_1608Metric" H 7130 1660 50  0001 C CNN
-F 3 "~" H 7130 1660 50  0001 C CNN
-	1    7130 1660
-	0    1    1    0
-$EndComp
-$Comp
 L Device:R_Small R7
 U 1 1 5C18291B
-P 7130 1935
-F 0 "R7" V 6934 1935 50  0000 C CNN
-F 1 "470" V 7025 1935 50  0000 C CNN
-F 2 "Resistor_SMD:R_0603_1608Metric" H 7130 1935 50  0001 C CNN
-F 3 "~" H 7130 1935 50  0001 C CNN
-	1    7130 1935
-	0    1    1    0
+P 7685 1360
+F 0 "R7" V 7489 1360 50  0000 C CNN
+F 1 "470" V 7580 1360 50  0000 C CNN
+F 2 "Resistor_SMD:R_0603_1608Metric" H 7685 1360 50  0001 C CNN
+F 3 "~" H 7685 1360 50  0001 C CNN
+	1    7685 1360
+	0    -1   -1   0
 $EndComp
 $Comp
 L Device:R_Small R8
 U 1 1 5C18296B
-P 7130 2210
-F 0 "R8" V 6934 2210 50  0000 C CNN
-F 1 "470" V 7025 2210 50  0000 C CNN
-F 2 "Resistor_SMD:R_0603_1608Metric" H 7130 2210 50  0001 C CNN
-F 3 "~" H 7130 2210 50  0001 C CNN
-	1    7130 2210
-	0    1    1    0
-$EndComp
-$Comp
-L Device:LED D1
-U 1 1 5C182A41
-P 7555 1660
-F 0 "D1" H 7546 1876 50  0000 C CNN
-F 1 "CAPS" H 7546 1785 50  0000 C CNN
-F 2 "LED_THT:LED_D1.8mm_W3.3mm_H2.4mm" H 7555 1660 50  0001 C CNN
-F 3 "~" H 7555 1660 50  0001 C CNN
-	1    7555 1660
-	1    0    0    -1
-$EndComp
-$Comp
-L Device:LED D2
-U 1 1 5C182B17
-P 7555 1935
-F 0 "D2" H 7546 2151 50  0000 C CNN
-F 1 "Num" H 7546 2060 50  0000 C CNN
-F 2 "LED_THT:LED_D1.8mm_W3.3mm_H2.4mm" H 7555 1935 50  0001 C CNN
-F 3 "~" H 7555 1935 50  0001 C CNN
-	1    7555 1935
-	1    0    0    -1
-$EndComp
-$Comp
-L Device:LED D3
-U 1 1 5C182B6D
-P 7555 2210
-F 0 "D3" H 7546 2426 50  0000 C CNN
-F 1 "Scroll" H 7546 2335 50  0000 C CNN
-F 2 "LED_THT:LED_D1.8mm_W3.3mm_H2.4mm" H 7555 2210 50  0001 C CNN
-F 3 "~" H 7555 2210 50  0001 C CNN
-	1    7555 2210
-	1    0    0    -1
-$EndComp
-Text GLabel 7880 1660 2    50   Input ~ 0
+P 7685 1635
+F 0 "R8" V 7489 1635 50  0000 C CNN
+F 1 "470" V 7580 1635 50  0000 C CNN
+F 2 "Resistor_SMD:R_0603_1608Metric" H 7685 1635 50  0001 C CNN
+F 3 "~" H 7685 1635 50  0001 C CNN
+	1    7685 1635
+	0    -1   -1   0
+$EndComp
+Text GLabel 6935 1085 0    50   Input ~ 0
 Caps
-Text GLabel 7880 1935 2    50   Input ~ 0
+Text GLabel 6935 1360 0    50   Input ~ 0
 Num
-Text GLabel 7880 2210 2    50   Input ~ 0
+Text GLabel 6935 1635 0    50   Input ~ 0
 Scrl
 Wire Wire Line
-	7705 1660 7880 1660
-Wire Wire Line
-	7705 1935 7880 1935
-Wire Wire Line
-	7705 2210 7880 2210
-Wire Wire Line
-	7405 2210 7230 2210
-Wire Wire Line
-	7405 1935 7230 1935
-Wire Wire Line
-	7405 1660 7230 1660
+	7410 1635 7585 1635
+Wire Wire Line
+	7410 1360 7585 1360
 $Comp
 L power:GND #PWR0116
 U 1 1 5C19F14D
-P 6880 1610
-F 0 "#PWR0116" H 6880 1360 50  0001 C CNN
-F 1 "GND" H 6885 1437 50  0000 C CNN
-F 2 "" H 6880 1610 50  0001 C CNN
-F 3 "" H 6880 1610 50  0001 C CNN
-	1    6880 1610
-	-1   0    0    1
-$EndComp
-Wire Wire Line
-	6880 1610 6880 1660
-Wire Wire Line
-	6880 2210 7030 2210
-Wire Wire Line
-	7030 1660 6880 1660
-Connection ~ 6880 1660
-Wire Wire Line
-	6880 1660 6880 1935
-Wire Wire Line
-	7030 1935 6880 1935
-Connection ~ 6880 1935
-Wire Wire Line
-	6880 1935 6880 2210
+P 7935 1685
+F 0 "#PWR0116" H 7935 1435 50  0001 C CNN
+F 1 "GND" H 7940 1512 50  0000 C CNN
+F 2 "" H 7935 1685 50  0001 C CNN
+F 3 "" H 7935 1685 50  0001 C CNN
+	1    7935 1685
+	1    0    0    -1
+$EndComp
 $Sheet
 S 9075 4940 1325 1000
@@
 Wire Wire Line
 	3670 1570 3715 1570
+Wire Wire Line
+	7935 1635 7785 1635
+Wire Wire Line
+	7785 1360 7935 1360
+Wire Wire Line
+	7110 1635 6935 1635
+Wire Wire Line
+	7110 1360 6935 1360
+Wire Wire Line
+	7110 1085 6935 1085
+$Comp
+L Device:LED D3
+U 1 1 5C182B6D
+P 7260 1635
+F 0 "D3" H 7251 1851 50  0000 C CNN
+F 1 "Scroll" H 7251 1760 50  0000 C CNN
+F 2 "LED_THT:LED_D1.8mm_W3.3mm_H2.4mm" H 7260 1635 50  0001 C CNN
+F 3 "~" H 7260 1635 50  0001 C CNN
+	1    7260 1635
+	-1   0    0    1
+$EndComp
+$Comp
+L Device:LED D2
+U 1 1 5C182B17
+P 7260 1360
+F 0 "D2" H 7251 1576 50  0000 C CNN
+F 1 "Num" H 7251 1485 50  0000 C CNN
+F 2 "LED_THT:LED_D1.8mm_W3.3mm_H2.4mm" H 7260 1360 50  0001 C CNN
+F 3 "~" H 7260 1360 50  0001 C CNN
+	1    7260 1360
+	-1   0    0    1
+$EndComp
+$Comp
+L Device:LED D1
+U 1 1 5C182A41
+P 7260 1085
+F 0 "D1" H 7251 1301 50  0000 C CNN
+F 1 "CAPS" H 7251 1210 50  0000 C CNN
+F 2 "LED_THT:LED_D1.8mm_W3.3mm_H2.4mm" H 7260 1085 50  0001 C CNN
+F 3 "~" H 7260 1085 50  0001 C CNN
+	1    7260 1085
+	-1   0    0    1
+$EndComp
+Wire Wire Line
+	7935 1685 7935 1635
+Wire Wire Line
+	7410 1085 7585 1085
+Wire Wire Line
+	7785 1085 7935 1085
+$Comp
+L Device:R_Small R6
+U 1 1 5C1827C5
+P 7685 1085
+F 0 "R6" V 7489 1085 50  0000 C CNN
+F 1 "470" V 7580 1085 50  0000 C CNN
+F 2 "Resistor_SMD:R_0603_1608Metric" H 7685 1085 50  0001 C CNN
+F 3 "~" H 7685 1085 50  0001 C CNN
+	1    7685 1085
+	0    -1   -1   0
+$EndComp
+Connection ~ 7935 1360
+Wire Wire Line
+	7935 1360 7935 1085
+Connection ~ 7935 1635
+Wire Wire Line
+	7935 1635 7935 1360
+$Comp
+L transistors:MMBT3904 Q1
+U 1 1 5E9E999A
+P 5390 4995
+F 0 "Q1" H 5581 5041 50  0000 L CNN
+F 1 "MMBT3904" H 5581 4950 50  0000 L CNN
+F 2 "Package_TO_SOT_SMD:SOT-23" H 5590 4920 50  0001 L CIN
+F 3 "https://www.fairchildsemi.com/datasheets/2N/2N3904.pdf" H 5390 4995 50  0001 L CNN
+	1    5390 4995
+	1    0    0    -1
+$EndComp
 $EndSCHEMATC

Commit message: Added base for Rev 6
Parts:
- removed C8: 1uf, Capacitor_SMD:C_0603_1608Metric, symbol Device:C_Small
- removed D1: CAPS, LED_THT:LED_D1.8mm_W3.3mm_H2.4mm, symbol Device:LED
- removed D2: Num, LED_THT:LED_D1.8mm_W3.3mm_H2.4mm, symbol Device:LED
- removed D3: Scroll, LED_THT:LED_D1.8mm_W3.3mm_H2.4mm, symbol Device:LED
- removed J2: AVR-ISP-6, Connector_PinHeader_2.54mm:PinHeader_2x03_P2.54mm_Vertical, symbol Connector:AVR-ISP-6
- removed Q1: MMBT3904, Package_TO_SOT_SMD:SOT-23, symbol transistors:MMBT3904
- removed R3: 10k, Resistor_SMD:R_0603_1608Metric, symbol Device:R_Small
- removed R4: 10K, Resistor_SMD:R_0603_1608Metric, symbol Device:R_Small
- removed R6, R7, R8: 470, Resistor_SMD:R_0603_1608Metric, symbol Device:R_Small
- removed U1: ATmega32U4-MU, Package_DFN_QFN:QFN-44-1EP_7x7mm_P0.5mm_EP5.2x5.2mm, symbol MCU_Microchip_ATmega:ATmega32U4-MU
- removed U2: PRTR5V0U2X, PRTR5V0U2X:SOT143B, symbol ai03-locallib:PRTR5V0U2X
- removed Y1: 16Mhz, Crystal:Crystal_SMD_2520-4Pin_2.5x2.0mm, symbol Device:Crystal_GND24
- added D1, D2, D3: WS2812B, CrumpPrints:WS2812-2020, symbol LED:WS2812B
- added D91: D, Diode_SMD:D_0603_1608Metric, symbol Device:D
- added Q1: BC850, Package_TO_SOT_SMD:SOT-23, symbol Transistor_BJT:BC850
- added Q2: MMBT3904, Package_TO_SOT_SMD:SOT-23, symbol Transistor_BJT:MMBT3904
- added U1: STM32F072CBTx, Package_QFP:LQFP-48_7x7mm_P0.5mm, symbol MCU_ST_STM32F0:STM32F072CBTx
- added U2: PRTR5V0U2X, random-keyboard-parts:SOT143B, symbol random-keyboard-parts:PRTR5V0U2X
- added U3: LD3985G33R_TSOT23, Package_TO_SOT_SMD:TSOT-23-5, symbol Regulator_Linear:LD3985G33R_TSOT23
- C2: value 22pF -> 10nf
- C3: value 22pF -> 10uf
- C4: value 100nF -> 4.7uf
- F1: footprint Fuse:Fuse_0805_2012Metric -> Fuse:Fuse_0603_1608Metric
- R1: value 22R -> 1.5k
- R2: value 22R -> 30k
- SW1: footprint Connector_PinHeader_2.54mm:PinHeader_2x01_P2.54mm_Vertical -> reset:ResetShort
Connections:
- net +5V: now also D1.1 (VDD), D2.1 (VDD), D3.1 (VDD), U3.1 (VIN), U3.3 (INH); no longer C4.2, C5.2, C6.2, C7.2
- net Col0: now also U1.31 (PA10)
- net Col1: now also U1.30 (PA9)
- net Col2: now also U1.29 (PA8)
- net Col3: now also U1.27 (PB14)
- net Col4: now also U1.26 (PB13)
- net Col5: now also U1.25 (PB12)
- net Col6: now also U1.20 (PB2)
- net Col7: now also U1.19 (PB1)
- net Col8: now also U1.18 (PB0)
- net Col9: now also U1.15 (PA5)
- net D+: now also USB1.6 (DP1), USB1.8 (DP2), U1.33 (PA12), U2.2 (IO1); no longer R2.1
- net D-: now also USB1.5 (DN2), USB1.7 (DN1), U1.32 (PA11), U2.3 (IO2); no longer R1.1
- net GND: now also R2.2, D1.3 (VSS), D2.3 (VSS), D3.3 (VSS), Q1.2 (E), Q2.2 (E), U1.23 (VSS), U1.35 (VSS), U1.47 (VSS), U1.8 (VSSA), U2.1 (GND), U3.2 (GND); no longer SW1.1
- net LEDGND: now also Q2.3 (C)
- net Row0: now also U1.37 (PA14)
- net Row1: now also U1.38 (PA15)
- net Row2: now also U1.39 (PB3)
- net Row3: now also U1.22 (PB11)
- net Row4: now also U1.21 (PB10)
- net VCC: now also U2.4 (VCC)
- net at R5.1: now also Q2.1 (B)
- net at R5.2: now also U1.16 (PA6)
- net E6 renamed B15
- net B15: now also D1.2 (DOUT)
- net RESET: no longer names the net of SW1.2
- net RESET: now also R1.1, D91.2 (A)
- net XTAL1: no longer names the net of C2.1
- net XTAL1: now also U3.4 (BYP)
- net XTAL2 renamed BOOT0
- net BOOT0: now also R2.1, D91.1 (K), U1.44 (BOOT0)
- new net: Q1.1 (B), R1.2
- new net: D1.4 (DIN), D2.2 (DOUT)
- new net: D2.4 (DIN), D3.2 (DOUT)
- new net +3V3: C4.2, C5.2, C6.2, C7.2, SW1.1, U1.1 (VBAT), U1.24 (VDD), U1.36 (VDDIO2), U1.48 (VDD), U1.9 (VDDA), U3.5 (VOUT)
- new net Col10: U1.14 (PA4)
- new net Col11: U1.13 (PA3)
- new net Col12: U1.12 (PA2)
- new net Col13: U1.11 (PA1)
- new net Col14: U1.34 (PA13)
- new net Col15: U1.4 (PC15)
- new net Col16: U1.2 (PC13)
- new net Col17: U1.3 (PC14)
- new net Col18: U1.10 (PA0)
- new net LED_OUT: D3.4 (DIN), U1.28 (PB15)
- new net NRST: Q1.3 (C), U1.7 (NRST)
- no-connect marks 3 -> 11
Other:
- note added: "Breakout\n"
- note added: "Decoupling Capacitors\n"
- note added: "Indicator LEDs\n"
- note added: "LDO Voltage Regulator\n\n"
- note added: "Polyfuse\n"
- note added: "Reset Circuit\n"
- note added: "USB & ESD Protection\n"
- moved on the sheet: C1, C4, C5, C6, C7, J3, R28, R5, R96, USB1

Commit message: Rerouted, added render
Connections:
- net Col16: now also U1.3 (PC14); no longer U1.2 (PC13)
- net Col17: now also U1.2 (PC13); no longer U1.3 (PC14)
Changed lines of the file:
@@
 Text GLabel 2780 4755 0    50   Input ~ 0
 Col15
+Text GLabel 2780 4655 0    50   Input ~ 0
+Col16
 Text GLabel 2780 4555 0    50   Input ~ 0
-Col16
-Text GLabel 2780 4655 0    50   Input ~ 0
 Col17
 Text GLabel 4080 4955 2    50   Input ~ 0

Commit message: updated rev6
Parts:
- D91: value D -> 1N4148; footprint Diode_SMD:D_0603_1608Metric -> Diode_SMD:D_SOD-123
Changed lines of the file:
@@
 	1460 2050 1580 2050
-Wire Wire Line
-	1580 2050 1580 2150
 Wire Wire Line
 	1580 2160 2170 2160
@@
 Wire Wire Line
 	2170 2020 2170 1810
-Wire Wire Line
-	1460 2150 1580 2150
-Connection ~ 1580 2150
-Wire Wire Line
-	1580 2150 1580 2160
 NoConn ~ 1460 1750
 NoConn ~ 1460 1150
@@
 	1    0    0    -1
 $EndComp
-$Comp
-L Device:Polyfuse_Small F1
-U 1 1 5EB19D46
-P 4520 1540
-F 0 "F1" V 4315 1540 50  0000 C CNN
-F 1 "500ma" V 4406 1540 50  0000 C CNN
-F 2 "Fuse:Fuse_0603_1608Metric" H 4570 1340 50  0001 L CNN
-F 3 "~" H 4520 1540 50  0001 C CNN
-	1    4520 1540
-	0    1    1    0
-$EndComp
 Wire Notes Line
 	3720 575  3720 2550
@@
 Wire Notes Line
 	5355 575  3720 575
-Text Notes 4360 2530 0    50   Italic 0
-Polyfuse\n
-Wire Wire Line
-	4420 1540 4145 1540
-Wire Wire Line
-	4620 1540 4940 1540
-$Comp
-L power:VCC #PWR0101
-U 1 1 5EB35097
-P 4145 1540
-F 0 "#PWR0101" H 4145 1390 50  0001 C CNN
-F 1 "VCC" V 4163 1667 50  0000 L CNN
-F 2 "" H 4145 1540 50  0001 C CNN
-F 3 "" H 4145 1540 50  0001 C CNN
-	1    4145 1540
-	0    -1   -1   0
-$EndComp
-$Comp
-L power:+5V #PWR0105
-U 1 1 5EB36440
-P 4940 1540
-F 0 "#PWR0105" H 4940 1390 50  0001 C CNN
-F 1 "+5V" V 4955 1668 50  0000 L CNN
-F 2 "" H 4940 1540 50  0001 C CNN
-F 3 "" H 4940 1540 50  0001 C CNN
-	1    4940 1540
-	0    1    1    0
-$EndComp
 Wire Notes Line
 	5410 575  5410 2550
@@
 P 8120 2820
 F 0 "D91" H 8120 2604 50  0000 C CNN
-F 1 "D" H 8120 2695 50  0000 C CNN
-F 2 "Diode_SMD:D_0603_1608Metric" H 8120 2820 50  0001 C CNN
+F 1 "1N4148" H 8120 2695 50  0000 C CNN
+F 2 "Diode_SMD:D_SOD-123" H 8120 2820 50  0001 C CNN
 F 3 "~" H 8120 2820 50  0001 C CNN
 	1    8120 2820
@@
 Text GLabel 4080 4955 2    50   Input ~ 0
 Col18
+Wire Wire Line
+	1580 2150 1580 2160
+Wire Wire Line
+	1580 2050 1580 2150
+Connection ~ 1580 2150
+Wire Wire Line
+	1460 2150 1580 2150
+Text Notes 4360 2530 0    50   Italic 0
+Polyfuse\n
+$Comp
+L power:+5V #PWR0105
+U 1 1 5EB36440
+P 4940 1540
+F 0 "#PWR0105" H 4940 1390 50  0001 C CNN
+F 1 "+5V" V 4955 1668 50  0000 L CNN
+F 2 "" H 4940 1540 50  0001 C CNN
+F 3 "" H 4940 1540 50  0001 C CNN
+	1    4940 1540
+	0    1    1    0
+$EndComp
+$Comp
+L power:VCC #PWR0101
+U 1 1 5EB35097
+P 4145 1540
+F 0 "#PWR0101" H 4145 1390 50  0001 C CNN
+F 1 "VCC" V 4163 1667 50  0000 L CNN
+F 2 "" H 4145 1540 50  0001 C CNN
+F 3 "" H 4145 1540 50  0001 C CNN
+	1    4145 1540
+	0    -1   -1   0
+$EndComp
+Wire Wire Line
+	4620 1540 4940 1540
+Wire Wire Line
+	4420 1540 4145 1540
+$Comp
+L Device:Polyfuse_Small F1
+U 1 1 5EB19D46
+P 4520 1540
+F 0 "F1" V 4315 1540 50  0000 C CNN
+F 1 "500ma" V 4406 1540 50  0000 C CNN
+F 2 "Fuse:Fuse_0603_1608Metric" H 4570 1340 50  0001 L CNN
+F 3 "~" H 4520 1540 50  0001 C CNN
+	1    4520 1540
+	0    1    1    0
+$EndComp
 $EndSCHEMATC

Commit message: updated rev6
Parts:
- added C10, C8, C9: 100nf, Capacitor_SMD:C_0603_1608Metric, symbol Device:C_Small
Connections:
- net +5V: now also C10.2, C8.2, C9.2
- net Col3: now also U1.40 (PB4); no longer U1.27 (PB14)
- net Col4: now also U1.41 (PB5); no longer U1.26 (PB13)
- net Col5: now also U1.42 (PB6); no longer U1.25 (PB12)
- net GND: now also C10.1, C8.1, C9.1
Changed lines of the file:
@@
 Text GLabel 4080 5755 2    50   Input ~ 0
 Col2
-Text GLabel 2780 6355 0    50   Input ~ 0
+Text GLabel 2780 5355 0    50   Input ~ 0
 Col3
-Text GLabel 2780 6255 0    50   Input ~ 0
+Text GLabel 2780 5455 0    50   Input ~ 0
 Col4
-Text GLabel 2780 6155 0    50   Input ~ 0
+Text GLabel 2780 5555 0    50   Input ~ 0
 Col5
 Text GLabel 2780 5155 0    50   Input ~ 0
@@
 	9310 2605 11165 2605
 Wire Notes Line
-	11165 2605 11165 5600
-Wire Notes Line
-	11165 5600 9310 5600
-Wire Notes Line
-	9310 5600 9310 2605
+	11165 3015 11165 6010
+Wire Notes Line
+	11165 6000 9310 6000
+Wire Notes Line
+	9320 6000 9310 2605
 Text Notes 10125 2510 0    50   Italic 0
 Breakout\n
-Text Notes 9985 5570 0    50   Italic 0
+Text Notes 9985 5970 0    50   Italic 0
 Indicator LEDs\n
 Wire Notes Line
@@
 Wire Wire Line
 	10230 4630 9475 4630
-Wire Wire Line
-	9475 4630 9475 3805
 Connection ~ 9475 3805
 Wire Wire Line
@@
 $EndComp
 NoConn ~ 2780 5855
-NoConn ~ 2780 5355
-NoConn ~ 2780 5455
 NoConn ~ 2780 5755
 NoConn ~ 4080 5655
 NoConn ~ 2780 5655
-NoConn ~ 2780 5555
 Text GLabel 9930 4930 0    50   Input ~ 0
 LED_OUT
@@
 	0    1    1    0
 $EndComp
+NoConn ~ 2780 6155
+NoConn ~ 2780 6255
+NoConn ~ 2780 6355
+$Comp
+L Device:C_Small C8
+U 1 1 5EDBC859
+P 9875 5565
+F 0 "C8" H 9885 5635 50  0000 L CNN
+F 1 "100nf" H 9885 5485 50  0000 L CNN
+F 2 "Capacitor_SMD:C_0603_1608Metric" H 9875 5565 50  0001 C CNN
+F 3 "~" H 9875 5565 50  0001 C CNN
+	1    9875 5565
+	-1   0    0    1
+$EndComp
+$Comp
+L Device:C_Small C9
+U 1 1 5EDBDAFF
+P 10260 5565
+F 0 "C9" H 10270 5635 50  0000 L CNN
+F 1 "100nf" H 10270 5485 50  0000 L CNN
+F 2 "Capacitor_SMD:C_0603_1608Metric" H 10260 5565 50  0001 C CNN
+F 3 "~" H 10260 5565 50  0001 C CNN
+	1    10260 5565
+	-1   0    0    1
+$EndComp
+$Comp
+L Device:C_Small C10
+U 1 1 5EDBE225
+P 10695 5565
+F 0 "C10" H 10705 5635 50  0000 L CNN
+F 1 "100nf" H 10705 5485 50  0000 L CNN
+F 2 "Capacitor_SMD:C_0603_1608Metric" H 10695 5565 50  0001 C CNN
+F 3 "~" H 10695 5565 50  0001 C CNN
+	1    10695 5565
+	-1   0    0    1
+$EndComp
+Connection ~ 10985 5230
+Wire Wire Line
+	10985 5230 10985 5665
+Wire Wire Line
+	10985 5665 10695 5665
+Connection ~ 10260 5665
+Wire Wire Line
+	10260 5665 9875 5665
+Connection ~ 10695 5665
+Wire Wire Line
+	10695 5665 10260 5665
+Wire Wire Line
+	10695 5465 10260 5465
+Wire Wire Line
+	9475 3805 9475 4630
+Connection ~ 9875 5465
+Wire Wire Line
+	9875 5465 9475 5465
+Connection ~ 10260 5465
+Wire Wire Line
+	10260 5465 9875 5465
+Connection ~ 9475 4630
+Wire Wire Line
+	9475 4630 9475 5465
 $EndSCHEMATC
